File: esp32Layout1.brd (EAGLE design)
At the start: 28 x 56.6 mm, 37 parts, among them U1 ESP-WROOM-32, Y3 32.768kHz

Commit message: 2nd bno055 version, sent to JLC for production
Parts:
- removed C13, C14: 22pF, microbuilder:0805-NO
- removed C15: 0.1uF, microbuilder:0805-NO
- removed C16: 0.1uF, microbuilder:0805_10MGAP
- removed D3: 1n4148, microbuilder:SOD-323
- removed JP7: (no value), microbuilder:1X04_ROUND_76
- removed R18, R19, R20, R25: 10K, microbuilder:0805-NO
- removed R21, R22: 4.7K, microbuilder:0805-NO
- removed U$68: BNO055, microbuilder:BNO055
- removed Y3: 32.768kHz, microbuilder:CRYSTAL_8X3.8
- added BNO055: BNO055, Tim Parts:BNO055
- added C1, C4: 0.1uF, microbuilder:0805-NO
- added C2, C3: 22pF, microbuilder:0805-NO
- added C5, C6: .1uF, microbuilder:0805_10MGAP
- added R2, R8: 10k, SparkFun-Resistors:0603
- added R3, R4, R7: 10K, microbuilder:0805-NO
- added R5, R6: 4.7K, microbuilder:0805-NO
- added Y1: 32.768kHz, microbuilder:CRYSTAL_8X3.8
- moved C18 16.9 mm to (9.88, 24.3)
- moved R1 10.9 mm to (14.2, 38.5), turned to 270 degrees
- moved U$11 8.25 mm to (10.0, 35.0)
- moved U$9 7.28 mm to (10.0, 41.0)
- moved U$3 2.00 mm to (25.6, 32.1)
- moved DRIVE 2.00 mm to (17.4, 25.3)
- moved U$1 2.00 mm to (25.6, 28.5)
- moved U$2 2.00 mm to (25.6, 36.6)
- moved U$4 2.00 mm to (25.6, 23.8)
- moved WEAPON 2.00 mm to (17.4, 33.4)
- moved VREG 1.20 mm to (4.51, 24.2)
Connections:
- removed net I2CADDR_3V: JP7.4, R20.1, U$68.17
- removed net INT_3V: JP7.3, U$68.14
- removed net NRESET_3V: D3.A, R25.1, U$68.11
- removed net PS0_3V: JP7.1, R18.1, U$68.6
- removed net PS1_3V: JP7.2, R19.1, U$68.5
- removed net VCC: DRIVE.1, R1.2, U1.2, UART.1, WEAPON.1
- new net ADDSEL: BNO055.P17
- new net INT: BNO055.P14
- new net N$1: BNO055.P5, R3.2
- new net N$5: R2.2, WEAPON.3
- new net N$6: BNO055.P9, C1.2
- new net N$7: BNO055.P27, C2.1, Y1.P$4
- new net N$8: BNO055.P26, C3.1, Y1.P$1
- new net N$9: BNO055.P4, R7.2
- net 3.3V: now also BNO055.P28, BNO055.P3, C4.2, R1.2, R4.2, R5.2, R6.2, R7.1, U1.2, UART.1; no longer C16.2, R21.2, R22.2, R25.2, U$68.28, U$68.3, U$68.4
- net GND: now also BNO055.P10, BNO055.P11, BNO055.P15, BNO055.P16, BNO055.P18, BNO055.P2, BNO055.P25, BNO055.P6, C1.1, C2.2, C3.2, C4.1, C5.1, C6.1, R3.1, R4.1; no longer C13.1, C14.1, C15.1, C16.1, D3.C, R18.2, R19.2, R20.2, U$68.10, U$68.15, U$68.16, U$68.18, U$68.2, U$68.25
- net IO16: now also R8.1; no longer DRIVE.3
- net IO21: now also R2.1; no longer WEAPON.3
- net N$10: now also DRIVE.3, R8.2; no longer C13.2, U$68.27, Y3.P$4
- net N$11: now also C5.2, DRIVE.1; no longer C14.2, U$68.26, Y3.P$1
- net N$12: now also C6.2, WEAPON.1; no longer C15.2, U$68.9
- net PWM4: now also U1.18; no longer U1.28
- net SCL_3V: now also BNO055.P19, R5.1; no longer R22.1, U$68.19
- net SDA_3V: now also BNO055.P20, R6.1; no longer R21.1, U$68.20
Routing:
- net 3.3V: track 46.3 -> 125.1 mm, vias 2 -> 6
- net VCC: track 71.2 -> 0.00 mm, vias 1 -> 0
- net GND: track 145.7 -> 181.5 mm, vias 12 -> 1
- net SDA_3V: track 60.7 -> 30.1 mm, vias 4 -> 2
- net PS0_3V: track 26.2 -> 0.00 mm, vias 1 -> 0
- net IO33: track 73.0 -> 49.5 mm
- net PS1_3V: track 21.3 -> 0.00 mm, vias 1 -> 0
- net N$11: track 8.33 -> 26.8 mm
- net SCL_3V: track 47.5 -> 29.7 mm, vias 4 -> 2
- net INT_3V: track 17.3 -> 0.00 mm, vias 1 -> 0
- net N$5: track 0.00 -> 15.5 mm, vias 0 -> 2
- net N$9: track 0.00 -> 9.25 mm, vias 0 -> 2
- net PWM2: track 48.9 -> 39.7 mm
- net IO25: track 59.4 -> 68.6 mm, vias 2 -> 0
- net IO32: track 59.3 -> 50.2 mm
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Other:
- board text added: "3v3"
- board text removed: "ADR"
- board text removed: "INT"
- board text removed: "PS0"
- board text removed: "PS1"
- board text removed: "VCC"

Commit message: V2 working stuff
Parts:
- moved R3 11.6 mm to (20.8, 41.9), turned to 90 degrees
- moved R5 10.9 mm to (17.3, 52.8), turned to 90 degrees
- moved R6 9.91 mm to (15.5, 52.8), turned to 90 degrees
- moved R7 5.97 mm to (18.9, 41.9), turned to 90 degrees
- moved C4 2.00 mm to (24.0, 45.0)
Routing:
- net SCL_3V: track 29.7 -> 43.3 mm
- net SDA_3V: track 30.1 -> 39.2 mm
- net N$9: track 9.25 -> 2.39 mm, vias 2 -> 0
- net IO32: track 50.2 -> 55.9 mm
- net GND: track 181.5 -> 178.3 mm, vias 1 -> 5
- net N$8: track 6.90 -> 8.85 mm
- net N$6: track 3.64 -> 5.11 mm, vias 0 -> 2
- net 3.3V: track 125.1 -> 124.5 mm, vias 6 -> 4
- net N$7: track 7.43 -> 7.30 mm, vias 2 -> 0
Other:
- board text added: "V2.0"

Commit message: Version 2.1 offical OSH PARK release
Parts:
- added AD, NR, SCL, SDA: (no value), wirepad:SMD1,27-2,54
- added C7: 10 uF, microbuilder:0805-NO
- added R9: 4.7K, microbuilder:0805-NO
Connections:
- removed net IO16: R8.1, U1.27
- removed net IO21: R2.1, U1.33
- removed net N$11: C5.2, DRIVE.1
- removed net N$12: C6.2, WEAPON.1
- new net IO34: R2.1, U1.6
- new net IO35: R8.1, U1.7
- new net NRESET: BNO055.P11, NR.1, R4.1
- net 3.3V: now also C5.2, C6.2, DRIVE.1, WEAPON.1
- net 5.0V: now also C7.2
- net ADDSEL: now also AD.1, R9.1
- net GND: now also C7.1, R9.2; no longer BNO055.P11, R4.1
- net PWM4: now also U1.31; no longer U1.18
- net SCL_3V: now also SCL.1, U1.36; no longer U1.20
- net SDA_3V: now also SDA.1, U1.33; no longer U1.21
Routing:
- net 3.3V: track 124.5 -> 159.3 mm, vias 4 -> 6
- net IO35: track 0.00 -> 28.0 mm, vias 0 -> 2
- net N$11: track 26.8 -> 0.00 mm
- net IO34: track 0.00 -> 21.4 mm, vias 0 -> 2
- net IO21: track 21.2 -> 0.00 mm, vias 2 -> 0
- net IO16: track 19.2 -> 0.00 mm
- net SCL_3V: track 43.3 -> 62.0 mm
- net SDA_3V: track 39.2 -> 55.4 mm
- net GND: track 178.3 -> 191.5 mm, vias 5 -> 16
- net NRESET: track 0.00 -> 10.6 mm, vias 0 -> 1
- net ADDSEL: track 0.00 -> 10.1 mm, vias 0 -> 1
- net N$12: track 3.09 -> 0.00 mm
- net PWM4: track 24.0 -> 22.5 mm
Other:
- board text added: "+"
- board text added: "-"
- board text added: "V2.1"
- board text removed: "V2.0"
